File: pi-diode-trailcam/hardware/kicad/pi-diode-carrier.kicad_pcb (KiCad board)
At the start: 4 copper layers, 100 x 80 mm, 53 parts, among them J1 Micro-Fit-2P-Batt, J2 Micro-Fit-4P-Mag, J3 Micro-Fit-4P-Radar, J4 Micro-Fit-4P-Pi5, J5 USB-C-5V-5A, J6 DC-Barrel-2.1mm, J7 Micro-Fit-2P-Deice, Q1 AO3401A, Q2A AOD403, Q2B AOD403, Q3 AO3401A, Q4 MMBT2222A, Q5 MMBT2222A, U1 HT7533-1, U2 RP2040-Pico-Socket, U3 TPS54560BDDAR, U4 ADS1115IDGSR

Commit message: Remediate all 21 findings from the 16 Oct 2026 project quality assessment
Routing:
- added copper zone on In2.Cu, net +12V_RAW
- added copper zone on In2.Cu, net +3V3_ALWAYS_ON
- added copper zone on In2.Cu, net +3V3_SENSORS
- added copper zone on In1.Cu, net GND
Changed lines of the file:
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@@
   (via (at 26.750 54.800) (size 0.65) (drill 0.35) (layers "F.Cu" "B.Cu") (net 1))
   (via (at 15.950 11.700) (size 0.65) (drill 0.35) (layers "F.Cu" "B.Cu") (net 1))
+  (zone (net 1) (net_name "GND") (layer "In1.Cu") (hatch edge 0.508)
+    (connect_pads (clearance 0.4))
+    (polygon (pts (xy 2.0 2.0) (xy 98.0 2.0) (xy 98.0 78.0) (xy 2.0 78.0)))
+  )
+  (zone (net 4) (net_name "+12V_RAW") (layer "In2.Cu") (hatch edge 0.508)
+    (connect_pads (clearance 0.4))
+    (polygon (pts (xy 6.0 66.0) (xy 34.0 66.0) (xy 34.0 78.0) (xy 6.0 78.0)))
+  )
+  (zone (net 6) (net_name "+3V3_ALWAYS_ON") (layer "In2.Cu") (hatch edge 0.508)
+    (connect_pads (clearance 0.4))
+    (polygon (pts (xy 42.0 22.0) (xy 95.0 22.0) (xy 95.0 65.0) (xy 42.0 65.0)))
+  )
+  (zone (net 7) (net_name "+3V3_SENSORS") (layer "In2.Cu") (hatch edge 0.508)
+    (connect_pads (clearance 0.4))
+    (polygon (pts (xy 72.0 67.0) (xy 96.0 67.0) (xy 96.0 78.0) (xy 72.0 78.0)))
+  )
 )
